File: OpenCelluloid.kicad_pcb (KiCad board)
At the start: 4 copper layers, 106 parts, among them J1 Conn_01x04_Male, J10 Conn_01x03_Male, J11 Conn_02x02_Counter_Clockwise, J12 Conn_01x03_Male, J13 Conn_02x02_Counter_Clockwise, J14 Conn_02x04_Counter_Clockwise, J2 Conn_02x03_Counter_Clockwise, J3 Conn_02x02_Counter_Clockwise, J4 Conn_01x03_Male, J5 Conn_01x02_Male, J6 ConnectorACMotor, J7 ConnectorMotorUpdated, J8 MS, J9 Conn_01x03_Male, Q1 IRF5305-Reverse-Polarity, Q2 IRF540N, Q3 IRF540N, Q4 IRF540N, Q5 IRF540N, Q6 IRF540N, Q7 IRF540N, Q8 BC847, SW1 powerButtonConnector, U1 POTENTIOMETER-OpenSourceCellu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, U10 IR2136, U11 Connector-Sensor, U12 stepStick, U13 PEC12R-ENCODER, U14 QRE1113, U15 74HC14, U16 Bridgelux-Vero-29-mech-ariadne, U17 ariadne-rescue_Noctua-NF-A4x1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, U18 ariadne-rescue_Noctua-NF-A4x1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, U2 POWER_CONNECTOR-DCJ250-20-B-K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, U3 Connector-LED, U4 OKI-78SR-3.3v, U5 OKI-78SR-5v, U6 OKI-78SR-12v, U7 LDH-45B-1050, U8 Connector-Sensor, U9 ESP32-WROOM-32D

Commit message: After pcb production
Parts:
- removed U16: Bridgelux-Vero-29-mech-ariadne, ariadne:Vero-29
- removed U17: ariadne-rescue_Noctua-NF-A4x10-Fan-mech-ariadne, ariadne:Noctua-NF-A4x10
- removed U18: ariadne-rescue_Noctua-NF-A4x10-Simple-Fan-ariadne, ariadne:Noctua-NF-A4x10
- removed U3: Connector-LED, Connector_JST:JST_PH_B2B-PH-K_1x02_P2.00mm_Vertical
- added J15: Conn_01x04_MountingPin, Connector_Molex:Molex_Micro-Fit_3.0_43650-0400_1x04_P3.00mm_Horizontal, F.Cu at (297.9, 111.1)
- added J16: Conn_01x04_MountingPin, ariadne:Vero29_w_Fan, F.Cu at (389.9, 205.9)
- added REF**: MountingHole_2.5mm_Pad_Via, MountingHole:MountingHole_2.5mm_Pad_Via, F.Cu at (353.5, 269.5)
- added REF**: MountingHole_3mm_Pad_Via, MountingHole:MountingHole_3mm_Pad_Via, F.Cu at (356.2, 238.0)
- added REF**: MountingHole_3mm_Pad_Via, MountingHole:MountingHole_3mm_Pad_Via, F.Cu at (194.0, 237.5)
- added REF**: MountingHole_3mm_Pad_Via, MountingHole:MountingHole_3mm_Pad_Via, F.Cu at (194.2, 196.5)
- added REF**: MountingHole_3mm_Pad_Via, MountingHole:MountingHole_3mm_Pad_Via, F.Cu at (355.2, 196.8)
- added REF**: MountingHole_3mm_Pad_Via, MountingHole:MountingHole_3mm_Pad_Via, F.Cu at (194.5, 107.0)
- added REF**: MountingHole_3mm_Pad_Via, MountingHole:MountingHole_3mm_Pad_Via, F.Cu at (355.8, 106.8)
- moved R24 370.7 mm to (273.2, 124.7), turned to 90 degrees
- moved R29 368.1 mm to (276.3, 124.7), turned to 90 degrees
- moved R16 273.5 mm to (342.9, 154.9), turned to 180 degrees
- moved U14 269.1 mm to (355.6, 262.3), turned to 270 degrees
- moved R23 264.1 mm to (356.9, 258.5), turned to 180 degrees
- moved R25 258.8 mm to (356.9, 254.7), turned to 180 degrees
- moved J10 248.6 mm to (350.5, 248.3), turned to 0 degrees
- moved D3 91.7 mm to (266.0, 173.0), turned to 270 degrees
- moved C6 13.7 mm to (309.0, 157.0)
- moved 50V-10uF1 11.9 mm to (295.7, 115.6)
- renumbered Murata-Ceramic-Capacitor-50v1-22uF3 to 50V-10uF1
Connections:
- U10 pad 10: EN -> EN2
- U9 pad 27: Net-(U9-Pad27) -> EN2
Routing:
- net +3V3: track 0.00 -> 430.4 mm, vias 0 -> 5
- net coilA: track 0.00 -> 391.3 mm, vias 0 -> 1
- net GNDD: track 0.00 -> 385.5 mm, vias 0 -> 9
- net +5V: track 0.00 -> 375.8 mm, vias 0 -> 9
- net coilB: track 0.00 -> 274.5 mm, vias 0 -> 4
- net GND: track 0.00 -> 272.1 mm, vias 0 -> 4
- net coilC: track 0.00 -> 257.6 mm, vias 0 -> 4
- net +24V: track 0.00 -> 241.0 mm, vias 0 -> 7
- net Net-(C1-Pad2): track 0.00 -> 216.8 mm
- net _ENCO-BUTTON: track 0.00 -> 204.7 mm
- net +12V: track 0.00 -> 186.2 mm, vias 0 -> 1
- net _CHANNEL-A: track 0.00 -> 185.0 mm
- net 45B_OUT-: track 0.00 -> 173.5 mm
- net _SENSOR: track 0.00 -> 158.3 mm, vias 0 -> 1
- net _CHANNEL-B: track 0.00 -> 151.8 mm, vias 0 -> 4
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- added copper zone on B.Cu, net (none)
- added copper zone on F.Cu, net (none)
- added copper zone on VCC, net +24V
- added copper zone on GND+GNDD, net GND
- added copper zone on GND+GNDD, net GNDD
Other:
- board outline added: 229.8 x 191 mm
- net class Power: trace_width 2 -> 1.5
- board text added: "Be like the promontory against which the waves continually break, but it stands firm and tames the fury of the water around it."
- board text added: "Look within. Within is the fountain of good, and it will ever bubble up, if thou wilt ever dig."
