File: OpenCelluloid.sch (KiCad schematic (older format))
At the start: 103 parts, among them J1 Conn_01x04_Male, J10 Conn_01x03_Male, J11 Conn_02x02_Counter_Clockwise, J12 Conn_02x03_Counter_Clockwise, J2 Conn_02x03_Counter_Clockwise, J3 Conn_02x02_Counter_Clockwise, J4 Conn_01x03_Male, J5 Conn_01x02_Male, J6 ConnectorACMotor, J7 ConnectorMotorUpdated, J8 MS, J9 Conn_01x03_Male, Q1 IRF5305-Reverse-Polarity, Q2 IRF540N, Q3 IRF540N, Q4 IRF540N, Q5 IRF540N, Q6 IRF540N, Q7 IRF540N, Q8 BC847, SW1 powerButtonConnector, U1 POTENTIOMETER-OpenSourceCellu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, U10 IR2136, U11 Connector-Sensor, U12 stepStick, U13 PEC12R-ENCODER, U14 QRE1113, U15 74HC14, U16 74HC14, U17 74HC14, U2 POWER_CONNECTOR-DCJ250-20-B-K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, U3 Connector-LED, U4 OKI-78SR-3.3v, U5 OKI-78SR-5v, U6 OKI-78SR-12v, U7 LDH-45B-1050, U8 Connector-Sensor, U9 ESP32-WROOM-32D

Commit message: 29.04
Parts:
- removed J12: Conn_02x03_Counter_Clockwise, Connector_PinHeader_2.54mm:PinHeader_2x03_P2.54mm_Vertical, symbol Connector_Generic:Conn_02x03_Counter_Clockwise
- added J12: Conn_01x03_Male, Connector_JST:JST_XH_B3B-XH-A_1x03_P2.50mm_Vertical, symbol Connector:Conn_01x03_Male
- added J13: Conn_02x02_Counter_Clockwise, knownParts:PinSocket_2x02_P2.54mm_Vertical_CounterClockWise, symbol Connector_Generic:Conn_02x02_Counter_Clockwise
- added J14: Conn_02x04_Counter_Clockwise, knownParts:PinHeader_2x04_P2.54mm_Vertical-CounterClowckWise, symbol Connector_Generic:Conn_02x04_Counter_Clockwise
- added unit 7 of U15
- added U16: Bridgelux-Vero-29-mech-ariadne, ariadne:Vero-29, symbol ariadne-rescue:Bridgelux-Vero-29-mech-ariadne
- added U17: ariadne-rescue_Noctua-NF-A4x10-Fan-mech-ariadne, ariadne:Noctua-NF-A4x10, symbol ariadne-v3-cache:ariadne-rescue_Noctua-NF-A4x10-Fan-mech-ariadne
- added U18: ariadne-rescue_Noctua-NF-A4x10-Simple-Fan-ariadne, ariadne:Noctua-NF-A4x10, symbol ariadne-v3-cache:ariadne-rescue_Noctua-NF-A4x10-Simple-Fan-ariadne
- C10, C9: footprint (none) -> Capacitor_THT:C_Rect_L7.0mm_W3.5mm_P5.00mm
- J11: footprint Connector_PinHeader_2.54mm:PinHeader_2x02_P2.54mm_Vertical -> knownParts:PinSocket_2x02_P2.54mm_Vertical_CounterClockWise
- J2: footprint Connector_PinHeader_2.54mm:PinHeader_2x03_P2.54mm_Vertical -> knownParts:PinHeader_2x03_P2.54mm_Vertical-CounterClockWise
- J3: footprint (none) -> knownParts:PinSocket_2x02_P2.54mm_Vertical_CounterClockWise
- Q2, Q3, Q4, Q5, Q6, Q7: footprint Package_TO_SOT_THT:TO-220-3_Vertical -> Package_TO_SOT_THT:TO-220-3_Horizontal_TabDown
- U1: footprint (none) -> OpenCelluloid:PDB12-H4301-Potentiometer
- U15: footprint (none) -> Package_DIP:DIP-14_W7.62mm_Socket
- U15: renamed from U16; footprint (none) -> Package_DIP:DIP-14_W7.62mm_Socket
- U15: renamed from U17; footprint (none) -> Package_DIP:DIP-14_W7.62mm_Socket
- renumbered Murata-Ceramic-Capacitor-50v1-22uF3 to 50V-10uF
Connections:
- net +12V: now also U18.2 (12V)
- net +3V3: now also J13.4 (Pin_4), U15.14 (VCC)
- net +5V: now also J13.3 (Pin_3)
- net GND: now also U18.1 (GND)
- net GNDD: now also J12.3 (Pin_3), U15.7 (GND)
- net SENSOR-CRASS: now also J14.1 (Pin_1)
- net SENSOR-SIMPLE: now also J14.2 (Pin_2)
- net SENSOR-SYNKINO: now also J14.3 (Pin_3)
- net _SENSOR: now also J14.5 (Pin_5), J14.6 (Pin_6), J14.7 (Pin_7), J14.8 (Pin_8)
- net at Q8.3 (C), R24.1, R26.1: now also U15.3; no longer U15.1
- net at R28.2: now also U15.4; no longer U15.2
- net at C10.2, R28.1: now also U15.5; no longer U15.1
- net at J11.2 (Pin_2), R29.2: now also U15.6; no longer U15.2
- new net: J12.1 (Pin_1), J13.1 (Pin_1), J13.2 (Pin_2)
- new net _SENSOR-SIGNAL: J12.2 (Pin_2), J14.4 (Pin_4)

Commit message: After pcb production
Parts:
- removed U16: Bridgelux-Vero-29-mech-ariadne, ariadne:Vero-29, symbol ariadne-rescue:Bridgelux-Vero-29-mech-ariadne
- removed U17: ariadne-rescue_Noctua-NF-A4x10-Fan-mech-ariadne, ariadne:Noctua-NF-A4x10, symbol ariadne-v3-cache:ariadne-rescue_Noctua-NF-A4x10-Fan-mech-ariadne
- removed U18: ariadne-rescue_Noctua-NF-A4x10-Simple-Fan-ariadne, ariadne:Noctua-NF-A4x10, symbol ariadne-v3-cache:ariadne-rescue_Noctua-NF-A4x10-Simple-Fan-ariadne
- removed U3: Connector-LED, Connector_JST:JST_PH_B2B-PH-K_1x02_P2.00mm_Vertical, symbol ariadne-rescue:Connector-LED-ariadne
- added J15: Conn_01x04_MountingPin, Connector_Molex:Molex_Micro-Fit_3.0_43650-0400_1x04_P3.00mm_Horizontal, symbol Connector_Generic_MountingPin:Conn_01x04_MountingPin
- added J16: Conn_01x04_MountingPin, ariadne:Vero29_w_Fan, symbol Connector_Generic_MountingPin:Conn_01x04_MountingPin
- renumbered 50V-10uF to 50V-10uF1
Connections:
- net +12V: now also J15.3 (Pin_3)
- net 45B_OUT+: now also J15.1 (Pin_1)
- net 45B_OUT-: now also J15.2 (Pin_2)
- net EN: no longer U10.10 (EN)
- net GND: now also J15.4 (Pin_4)
- net EN2: now reaches U9.27 (RX0)
- net EN2: now also U10.10 (EN)
Other:
- moved on the sheet: U1, U7
